Commit message: Removed basket

File: helpers/turtlebot/turtlebot3_waffle.urdf.xacro (robot description, xacro)
@@ -219,5 +219,8 @@
      <origin xyz="-0.15 -0.15 0.007" rpy="0 0 0"/>
      <geometry>
-       <mesh filename="package://turtlebot3_description/meshes/basket/basket.dae" scale="1 1 0.5"/>
+    <cylinder>
+    <radius>0.0001</radius>
+    <length>0.0001</length>
+ </cylinder>
      </geometry>
     </visual>
@@ -225,5 +228,8 @@
       <origin xyz="-0.15 -0.15 0.007" rpy="0 0 0"/>
      <geometry>
-       <mesh filename="package://turtlebot3_description/meshes/basket/basket.dae" scale="1 1 0.5"/>
+      <cylinder>
+    <radius>0.0001</radius>
+    <length>0.0001</length>
+ </cylinder>
      </geometry>
       <surface>
